Commit message: feat: demo moveit+rviz

File: maneuver_bringup/urdf/drone.urdf (robot description, URDF)
Before this commit: robot drone, 3 links, 2 joints
Links:
- removed link world
- link prop1: mass 0.01 -> None
Joints:
- removed joint world_to_base
- joint prop1_joint: origin xyz=0.3 0.3 0 rpy=0 0 0 -> xyz=0.3 0.3 0
